Commit message: add animation

File: src/urdf/4dof_2.urdf (robot description, URDF)
Before this commit: robot 4DOF_Robot, 13 links, 11 joints
Joints:
- joint fixed: origin xyz=1 1 0 rpy=0 0 -1.57 -> xyz=0.8 0.8 0 rpy=0 0 -1.57
- joint j1: origin xyz=0 0 0.4 rpy=0 0 0 -> xyz=0 0 0.2 rpy=0 0 0
- joint j1_2: origin xyz=0 0 0.4 rpy=0 0 0 -> xyz=0 0 0.2 rpy=0 0 0
- joint j3: origin xyz=0.4 0 0 rpy=0 0 1.57 -> xyz=0.5 0 0 rpy=0 0 2.36
- joint j3_2: origin xyz=0.4 0 0 rpy=0 0 1.57 -> xyz=0.5 0 0 rpy=0 0 2.36
- joint j4: origin xyz=0.3 0 0 rpy=0 0 -1.57 -> xyz=0.4 0 0 rpy=0 0 -1.57
- joint j4_2: origin xyz=0.3 0 0 rpy=0 0 -1.57 -> xyz=0.4 0 0 rpy=0 0 -1.57
- joint j5: origin xyz=0.2 0 0 rpy=0 0 0 -> xyz=0.3 0 0 rpy=0 0 0
- joint j5_2: origin xyz=0.2 0 0 rpy=0 0 0 -> xyz=0.3 0 0 rpy=0 0 0
